File: consoles.sch (KiCad schematic (older format))
At the start: 1 part

Commit message: Work so far.
Parts:
- added J4101: usbc-16p, usbc16p:usbc16p, symbol usbc-16p:usbc-16p
- U4101: renamed from U?; footprint (none) -> Package_DFN_QFN:QFN-64-1EP_9x9mm_P0.5mm_EP4.7x4.7mm_ThermalVias
Connections:
- net console_queen/usb_dn: now reaches U4101.1 (USBDN1_DM/PRT_DIS_M1)
- net console_drone3/usb_dn: now reaches U4101.11 (USBDN5_DM/PRTD_IS_M5)
- net console_drone3/usb_dp: now reaches U4101.12 (USBDN5_DP/PRT_DSI_P5)
- net console_queen/usb_dp: now reaches U4101.2 (USBDN1_DP/PRT_DIS_P1)
- net console_drone0/usb_dn: now reaches U4101.3 (USBDN2_DM/PRT_DIS_M2)
- net console_drone0/usb_dp: now reaches U4101.4 (USBDN2_DP/PRT_DIS_P2)
- net console_drone4/usb_dn: now reaches U4101.53 (USBDN6_DM/PRT_DIS_M6)
- net console_drone4/usb_dp: now reaches U4101.54 (USBDN6_DP/PRT_DIS_P6)
- net console_drone5/usb_dn: now reaches U4101.55 (USBDN7_DM/PRT_DIS_M7)
- net console_drone5/usb_dp: now reaches U4101.56 (USBDN7_DP/PRT_DIS_P7)
- net at U4101.58 (USBUP_DM): now also J4101.a7 (dn1), J4101.b7 (dn2)
- net at U4101.59 (USBUP_DP): now also J4101.a6 (dp1), J4101.b6 (dp2)
- net console_drone1/usb_dn: now reaches U4101.6 (USBDN3_DM/PRT_DIS_M3)
- net GND: now reaches U4101.65 (GND)
- net console_drone1/usb_dp: now reaches U4101.7 (USBDN3_DP/PRT_DIS_P3)
- net console_drone2/usb_dn: now reaches U4101.8 (USBDN4_DM/PRTD_IS_M4)
- net console_drone2/usb_dp: now reaches U4101.9 (USBDN4_DP/PRT_DIS_P4)
- new net: J4101.a1 (gnd), J4101.a12 (gnd), J4101.b1 (gnd), J4101.b12 (gnd)
- new net: J4101.a4 (vbus), J4101.a9 (vbus), J4101.b4 (vbus), J4101.b9 (vbus)
Other:
- note added: "Reference base: 1000"
- note added: "Reference base: 1100"
- note added: "Reference base: 1200"
- note added: "Reference base: 1300"
- note added: "Reference base: 1400"
- note added: "Reference base: 1500"
- note added: "Reference base: 1600"
- note added: "Reference base: 1700"
