File: rtlswch.sch (KiCad schematic (older format))
At the start: 8 parts

Commit message: Work so far.
Parts:
- added C205, C206, C207, C208, C209, C210, C211, C212, C213, C214, C215, C216, C217, C218, C219, C220, C221, C222, C223: C, Capacitor_SMD:C_0402_1005Metric, symbol Device:C
- added D201: LED, LED_SMD:LED_0603_1608Metric, symbol Device:LED
- added FB201, FB202, FB203, FB204: Ferrite_Bead, Inductor_SMD:L_0402_1005Metric, symbol Device:Ferrite_Bead
- added R203: R, Resistor_SMD:R_0402_1005Metric, symbol Device:R
- added Y201: 25MHz, Crystal:Crystal_SMD_Abracon_ABM8G-4Pin_3.2x2.5mm, symbol Device:Crystal_GND24
- C201, C202, C203, C204: renamed from C?; footprint (none) -> Capacitor_SMD:C_0402_1005Metric
- J201: renamed from J?; footprint (none) -> hanrun:HR961160C
- R201, R202: renamed from R?; footprint (none) -> Resistor_SMD:R_0402_1005Metric
- U201: renamed from U?; footprint (none) -> Package_DFN_QFN:QFN-64-1EP_9x9mm_P0.5mm_EP6x6mm_ThermalVias
Connections:
- net labels added: analog_1v0, analog_3v3, drone0_rxn, drone0_rxp, drone0_txn, drone0_txp, drone1_rxn, drone1_rxp, drone1_txn, drone1_txp, drone2_rxn, drone2_rxp, drone2_txn, drone2_txp, drone3_rxn, drone3_rxp, drone3_txn, drone3_txp, drone4_rxn, drone4_rxp, drone4_txn, drone4_txp, drone5_rxn, drone5_rxp, drone5_txn, drone5_txp, pll_1v0, pll_3v3, queen_rxn, queen_rxp, queen_txn, queen_txp, sw_1v0
- net labels removed: +1V0, drone_0_rxp
- wire segments 89 -> 230
Other:
- note added: "Reference base: 2100"
- note added: "Reference base: 2200"
- note added: "Reference base: 2300"
- note added: "Reference base: 2400"
- note added: "Reference base: 2500"
- note added: "Reference base: 2600"
- note added: "Reference base: 2700"
