File: switch_drone_port.sch (KiCad schematic (older format))
At the start: 4 parts

Commit message: Work so far.
Parts:
- added D901: LED, LED_SMD:LED_0603_1608Metric, symbol Device:LED
- added R901: R, Resistor_SMD:R_0402_1005Metric, symbol Device:R
- C301, C302, C303, C304: renamed from C?; footprint (none) -> Capacitor_SMD:C_0402_1005Metric
Connections:
- net drone_txn: now reaches C301.1
- net drone_txp: now reaches C302.1
- net drone_rxn: now reaches C303.1
- net drone_rxp: now reaches C304.1
- new net: D901.2 (A), R901.1
- new net GND: D901.1 (K)
- new net led: R901.2
Other:
- moved on the sheet: C301, C302, C303, C304
Changed lines of the file:
@@
 $Descr A4 11693 8268
 encoding utf-8
-Sheet 6 9
+Sheet 3 48
 Title ""
 Date ""
@@
 $EndDescr
 $Comp
-L Device:C C?
+L Device:C C301
 U 1 1 5F1FE174
-P 4950 2850
-AR Path="/5F1249CD/5F1F9E16/5F1FE174" Ref="C?"  Part="1"
-AR Path="/5F1249CD/5F21EF03/5F1FE174" Ref="C?"  Part="1"
-AR Path="/5F1249CD/5F22A52D/5F1FE174" Ref="C?"  Part="1"
-AR Path="/5F1249CD/5F22FE6A/5F1FE174" Ref="C?"  Part="1"
-AR Path="/5F1249CD/5F23AD4A/5F1FE174" Ref="C?"  Part="1"
-AR Path="/5F1249CD/5F2462D5/5F1FE174" Ref="C?"  Part="1"
-F 0 "C?" V 4698 2850 50  0000 C CNN
-F 1 "C" V 4789 2850 50  0000 C CNN
-F 2 "" H 4988 2700 50  0001 C CNN
-F 3 "~" H 4950 2850 50  0001 C CNN
-	1    4950 2850
+P 1300 800
+AR Path="/5F1249CD/5F1F9E16/5F1FE174" Ref="C301"  Part="1"
+AR Path="/5F1249CD/5F21EF03/5F1FE174" Ref="C401"  Part="1"
+AR Path="/5F1249CD/5F22A52D/5F1FE174" Ref="C501"  Part="1"
+AR Path="/5F1249CD/5F22FE6A/5F1FE174" Ref="C601"  Part="1"
+AR Path="/5F1249CD/5F23AD4A/5F1FE174" Ref="C701"  Part="1"
+AR Path="/5F1249CD/5F2462D5/5F1FE174" Ref="C801"  Part="1"
+AR Path="/5F1249CD/5F431A31/5F1FE174" Ref="C901"  Part="1"
+F 0 "C301" V 1048 800 50  0000 C CNN
+F 1 "C" V 1139 800 50  0000 C CNN
+F 2 "Capacitor_SMD:C_0402_1005Metric" H 1338 650 50  0001 C CNN
+F 3 "~" H 1300 800 50  0001 C CNN
+	1    1300 800
 	0    1    1    0
 $EndComp
 $Comp
-L Device:C C?
+L Device:C C302
 U 1 1 5F1FE801
-P 4950 3250
-AR Path="/5F1249CD/5F1F9E16/5F1FE801" Ref="C?"  Part="1"
-AR Path="/5F1249CD/5F21EF03/5F1FE801" Ref="C?"  Part="1"
-AR Path="/5F1249CD/5F22A52D/5F1FE801" Ref="C?"  Part="1"
-AR Path="/5F1249CD/5F22FE6A/5F1FE801" Ref="C?"  Part="1"
-AR Path="/5F1249CD/5F23AD4A/5F1FE801" Ref="C?"  Part="1"
-AR Path="/5F1249CD/5F2462D5/5F1FE801" Ref="C?"  Part="1"
-F 0 "C?" V 4698 3250 50  0000 C CNN
-F 1 "C" V 4789 3250 50  0000 C CNN
-F 2 "" H 4988 3100 50  0001 C CNN
-F 3 "~" H 4950 3250 50  0001 C CNN
-	1    4950 3250
+P 1300 1200
+AR Path="/5F1249CD/5F1F9E16/5F1FE801" Ref="C302"  Part="1"
+AR Path="/5F1249CD/5F21EF03/5F1FE801" Ref="C402"  Part="1"
+AR Path="/5F1249CD/5F22A52D/5F1FE801" Ref="C502"  Part="1"
+AR Path="/5F1249CD/5F22FE6A/5F1FE801" Ref="C602"  Part="1"
+AR Path="/5F1249CD/5F23AD4A/5F1FE801" Ref="C702"  Part="1"
+AR Path="/5F1249CD/5F2462D5/5F1FE801" Ref="C802"  Part="1"
+AR Path="/5F1249CD/5F431A31/5F1FE801" Ref="C902"  Part="1"
+F 0 "C302" V 1048 1200 50  0000 C CNN
+F 1 "C" V 1139 1200 50  0000 C CNN
+F 2 "Capacitor_SMD:C_0402_1005Metric" H 1338 1050 50  0001 C CNN
+F 3 "~" H 1300 1200 50  0001 C CNN
+	1    1300 1200
 	0    1    1    0
 $EndComp
 $Comp
-L Device:C C?
+L Device:C C303
 U 1 1 5F1FED64
-P 4950 3650
-AR Path="/5F1249CD/5F1F9E16/5F1FED64" Ref="C?"  Part="1"
-AR Path="/5F1249CD/5F21EF03/5F1FED64" Ref="C?"  Part="1"
-AR Path="/5F1249CD/5F22A52D/5F1FED64" Ref="C?"  Part="1"
-AR Path="/5F1249CD/5F22FE6A/5F1FED64" Ref="C?"  Part="1"
-AR Path="/5F1249CD/5F23AD4A/5F1FED64" Ref="C?"  Part="1"
-AR Path="/5F1249CD/5F2462D5/5F1FED64" Ref="C?"  Part="1"
-F 0 "C?" V 4698 3650 50  0000 C CNN
-F 1 "C" V 4789 3650 50  0000 C CNN
-F 2 "" H 4988 3500 50  0001 C CNN
-F 3 "~" H 4950 3650 50  0001 C CNN
-	1    4950 3650
+P 1300 1600
+AR Path="/5F1249CD/5F1F9E16/5F1FED64" Ref="C303"  Part="1"
+AR Path="/5F1249CD/5F21EF03/5F1FED64" Ref="C403"  Part="1"
+AR Path="/5F1249CD/5F22A52D/5F1FED64" Ref="C503"  Part="1"
+AR Path="/5F1249CD/5F22FE6A/5F1FED64" Ref="C603"  Part="1"
+AR Path="/5F1249CD/5F23AD4A/5F1FED64" Ref="C703"  Part="1"
+AR Path="/5F1249CD/5F2462D5/5F1FED64" Ref="C803"  Part="1"
+AR Path="/5F1249CD/5F431A31/5F1FED64" Ref="C903"  Part="1"
+F 0 "C303" V 1048 1600 50  0000 C CNN
+F 1 "C" V 1139 1600 50  0000 C CNN
+F 2 "Capacitor_SMD:C_0402_1005Metric" H 1338 1450 50  0001 C CNN
+F 3 "~" H 1300 1600 50  0001 C CNN
+	1    1300 1600
 	0    1    1    0
 $EndComp
 $Comp
-L Device:C C?
+L Device:C C304
 U 1 1 5F1FF1E5
-P 4950 4050
-AR Path="/5F1249CD/5F1F9E16/5F1FF1E5" Ref="C?"  Part="1"
-AR Path="/5F1249CD/5F21EF03/5F1FF1E5" Ref="C?"  Part="1"
-AR Path="/5F1249CD/5F22A52D/5F1FF1E5" Ref="C?"  Part="1"
-AR Path="/5F1249CD/5F22FE6A/5F1FF1E5" Ref="C?"  Part="1"
-AR Path="/5F1249CD/5F23AD4A/5F1FF1E5" Ref="C?"  Part="1"
-AR Path="/5F1249CD/5F2462D5/5F1FF1E5" Ref="C?"  Part="1"
-F 0 "C?" V 4698 4050 50  0000 C CNN
-F 1 "C" V 4789 4050 50  0000 C CNN
-F 2 "" H 4988 3900 50  0001 C CNN
-F 3 "~" H 4950 4050 50  0001 C CNN
-	1    4950 4050
+P 1300 2000
+AR Path="/5F1249CD/5F1F9E16/5F1FF1E5" Ref="C304"  Part="1"
+AR Path="/5F1249CD/5F21EF03/5F1FF1E5" Ref="C404"  Part="1"
+AR Path="/5F1249CD/5F22A52D/5F1FF1E5" Ref="C504"  Part="1"
+AR Path="/5F1249CD/5F22FE6A/5F1FF1E5" Ref="C604"  Part="1"
+AR Path="/5F1249CD/5F23AD4A/5F1FF1E5" Ref="C704"  Part="1"
+AR Path="/5F1249CD/5F2462D5/5F1FF1E5" Ref="C804"  Part="1"
+AR Path="/5F1249CD/5F431A31/5F1FF1E5" Ref="C904"  Part="1"
+F 0 "C304" V 1048 2000 50  0000 C CNN
+F 1 "C" V 1139 2000 50  0000 C CNN
+F 2 "Capacitor_SMD:C_0402_1005Metric" H 1338 1850 50  0001 C CNN
+F 3 "~" H 1300 2000 50  0001 C CNN
+	1    1300 2000
 	0    1    1    0
 $EndComp
-Text HLabel 4700 2850 0    50   Input ~ 0
+Text HLabel 1050 800  0    50   Input ~ 0
 switch_rxn
-Text HLabel 4700 3250 0    50   Input ~ 0
+Text HLabel 1050 1200 0    50   Input ~ 0
 switch_rxp
-Text HLabel 4700 3650 0    50   Input ~ 0
+Text HLabel 1050 1600 0    50   Input ~ 0
 switch_txn
-Text HLabel 4700 4050 0    50   Input ~ 0
+Text HLabel 1050 2000 0    50   Input ~ 0
 switch_txp
 Wire Wire Line
-	4700 2850 4800 2850
+	1050 800  1150 800
 Wire Wire Line
-	4700 3250 4800 3250
+	1050 1200 1150 1200
 Wire Wire Line
-	4700 3650 4800 3650
+	1050 1600 1150 1600
 Wire Wire Line
-	4700 4050 4800 4050
+	1050 2000 1150 2000
+Text HLabel 1550 1600 2    50   Input ~ 0
+drone_rxn
+Wire Wire Line
+	1450 800  1550 800
+Wire Wire Line
+	1450 1600 1550 1600
+Text HLabel 1550 2000 2    50   Input ~ 0
+drone_rxp
+Wire Wire Line
+	1550 2000 1450 2000
+Text HLabel 1550 1200 2    50   Input ~ 0
+drone_txp
+Wire Wire Line
+	1550 1200 1450 1200
+Text HLabel 1550 800  2    50   Input ~ 0
+drone_txn
+$Comp
+L Device:LED D901
+U 1 1 5FA32147
+P 1550 2650
+AR Path="/5F1249CD/5F431A31/5FA32147" Ref="D901"  Part="1"
+AR Path="/5F1249CD/5F1F9E16/5FA32147" Ref="D301"  Part="1"
+AR Path="/5F1249CD/5F21EF03/5FA32147" Ref="D401"  Part="1"
+AR Path="/5F1249CD/5F22A52D/5FA32147" Ref="D501"  Part="1"
+AR Path="/5F1249CD/5F22FE6A/5FA32147" Ref="D601"  Part="1"
+AR Path="/5F1249CD/5F23AD4A/5FA32147" Ref="D701"  Part="1"
+AR Path="/5F1249CD/5F2462D5/5FA32147" Ref="D801"  Part="1"
+F 0 "D301" V 1589 2532 50  0000 R CNN
+F 1 "LED" V 1498 2532 50  0000 R CNN
+F 2 "LED_SMD:LED_0603_1608Metric" H 1550 2650 50  0001 C CNN
+F 3 "~" H 1550 2650 50  0001 C CNN
+	1    1550 2650
+	0    -1   -1   0
+$EndComp
+$Comp
+L Device:R R901
+U 1 1 5FA32CFF
+P 1300 2450
+AR Path="/5F1249CD/5F431A31/5FA32CFF" Ref="R901"  Part="1"
+AR Path="/5F1249CD/5F1F9E16/5FA32CFF" Ref="R301"  Part="1"
+AR Path="/5F1249CD/5F21EF03/5FA32CFF" Ref="R401"  Part="1"
+AR Path="/5F1249CD/5F22A52D/5FA32CFF" Ref="R501"  Part="1"
+AR Path="/5F1249CD/5F22FE6A/5FA32CFF" Ref="R601"  Part="1"
+AR Path="/5F1249CD/5F23AD4A/5FA32CFF" Ref="R701"  Part="1"
+AR Path="/5F1249CD/5F2462D5/5FA32CFF" Ref="R801"  Part="1"
+F 0 "R301" V 1093 2450 50  0000 C CNN
+F 1 "R" V 1184 2450 50  0000 C CNN
+F 2 "Resistor_SMD:R_0402_1005Metric" V 1230 2450 50  0001 C CNN
+F 3 "~" H 1300 2450 50  0001 C CNN
+	1    1300 2450
+	0    1    1    0
+$EndComp
+Wire Wire Line
+	1450 2450 1550 2450
+Wire Wire Line
+	1550 2450 1550 2500
+$Comp
+L power:GND #PWR0901
+U 1 1 5FA33610
+P 1550 2900
+AR Path="/5F1249CD/5F431A31/5FA33610" Ref="#PWR0901"  Part="1"
+AR Path="/5F1249CD/5F1F9E16/5FA33610" Ref="#PWR0301"  Part="1"
+AR Path="/5F1249CD/5F21EF03/5FA33610" Ref="#PWR0401"  Part="1"
+AR Path="/5F1249CD/5F22A52D/5FA33610" Ref="#PWR0501"  Part="1"
+AR Path="/5F1249CD/5F22FE6A/5FA33610" Ref="#PWR0601"  Part="1"
+AR Path="/5F1249CD/5F23AD4A/5FA33610" Ref="#PWR0701"  Part="1"
+AR Path="/5F1249CD/5F2462D5/5FA33610" Ref="#PWR0801"  Part="1"
+F 0 "#PWR0901" H 1550 2650 50  0001 C CNN
+F 1 "GND" H 1555 2727 50  0000 C CNN
+F 2 "" H 1550 2900 50  0001 C CNN
+F 3 "" H 1550 2900 50  0001 C CNN
+	1    1550 2900
+	1    0    0    -1
+$EndComp
+Wire Wire Line
+	1550 2800 1550 2900
+Text HLabel 1050 2450 0    50   Input ~ 0
+led
+Wire Wire Line
+	1050 2450 1150 2450
 $EndSCHEMATC
